Commit message: feat: working example

File: src/walli_description/urdf/walliV2.urdf (robot description, URDF)
Before this commit: robot walliV2, 19 links, 18 joints
Links:
- removed link left_center_wheel
- removed link left_front_wheel
- removed link left_rear_wheel
- removed link leftbogie
- removed link leftrocker
- removed link right_center_wheel
- removed link right_front_wheel
- removed link right_rear_wheel
- removed link rightbogie
- removed link rightrocker
Joints:
- removed joint left_center_wheel_joint
- removed joint left_front_wheel_joint
- removed joint left_rear_wheel_joint
- removed joint leftbogiejoint
- removed joint leftrockerjoint
- removed joint right_center_wheel_joint
- removed joint right_front_wheel_joint
- removed joint right_rear_wheel_joint
- removed joint rightbogiejoint
- removed joint rightrockerjoint
